Commit message: Updated to Cogniteam's office map

File: mrm_sim/models/10robots.xacro (robot description, xacro)
@@ -4,13 +4,13 @@
        xmlns:interface="http://playerstage.sourceforge.net/gazebo/xmlschema/#interface"
        xmlns:xacro="http://playerstage.sourceforge.net/gazebo/xmlschema/#interface">
-<xacro:pioneer_model robot_id="1"  position="2 0 0.3 0 0 0" />
-<xacro:pioneer_model robot_id="2"  position="3 -11 0.3 0 0 0" />
-<xacro:pioneer_model robot_id="3"  position="17 -16 0.3 0 0 -3.1415" />
-<xacro:pioneer_model robot_id="4"  position="3 0 0.3 0 0 0" />
-<xacro:pioneer_model robot_id="5"  position="4 0 0.3 0 0 0" />
-<xacro:pioneer_model robot_id="6"  position="5 0 0.3 0 0 0" />
-<xacro:pioneer_model robot_id="7"  position="6 0 0.3 0 0 0" />
-<xacro:pioneer_model robot_id="8"  position="7 0 0.3 0 0 0" />
-<xacro:pioneer_model robot_id="9"  position="8 0 0.3 0 0 0" />
-<xacro:pioneer_model robot_id="10" position="9 0 0.3 0 0 0" />
+<xacro:pioneer_model robot_id="1"  position="1 1 0.3 0 0 0" />
+<xacro:pioneer_model robot_id="2"  position="2 1 0.3 0 0 0" />
+<xacro:pioneer_model robot_id="3"  position="3 1 0.3 0 0 0" />
+<xacro:pioneer_model robot_id="4"  position="1 2 0.3 0 0 0" />
+<xacro:pioneer_model robot_id="5"  position="2 2 0.3 0 0 0" />
+<xacro:pioneer_model robot_id="6"  position="3 2 0.3 0 0 0" />
+<xacro:pioneer_model robot_id="7"  position="1 3 0.3 0 0 0" />
+<xacro:pioneer_model robot_id="8"  position="2 3 0.3 0 0 0" />
+<xacro:pioneer_model robot_id="9"  position="3 3 0.3 0 0 0" />
+<xacro:pioneer_model robot_id="10" position="4 1 0.3 0 0 0" />
 </xacro>

File: mrm_sim/models/1robots.xacro (robot description, xacro)
@@ -4,4 +4,4 @@
        xmlns:interface="http://playerstage.sourceforge.net/gazebo/xmlschema/#interface"
        xmlns:xacro="http://playerstage.sourceforge.net/gazebo/xmlschema/#interface">
-<xacro:pioneer_model robot_id="1"  position="2 0 0.3 0 0 0" />
+<xacro:pioneer_model robot_id="1"  position="1 1 0.3 0 0 0" />
 </xacro>

File: mrm_sim/models/2robots.xacro (robot description, xacro)
@@ -4,5 +4,5 @@
        xmlns:interface="http://playerstage.sourceforge.net/gazebo/xmlschema/#interface"
        xmlns:xacro="http://playerstage.sourceforge.net/gazebo/xmlschema/#interface">
-<xacro:pioneer_model robot_id="1"  position="2 0 0.3 0 0 0" />
-<xacro:pioneer_model robot_id="2"  position="3 -11 0.3 0 0 0" />
+<xacro:pioneer_model robot_id="1"  position="1 1 0.3 0 0 0" />
+<xacro:pioneer_model robot_id="2"  position="2 1 0.3 0 0 0" />
 </xacro>

File: mrm_sim/models/3robots.xacro (robot description, xacro)
@@ -4,6 +4,6 @@
        xmlns:interface="http://playerstage.sourceforge.net/gazebo/xmlschema/#interface"
        xmlns:xacro="http://playerstage.sourceforge.net/gazebo/xmlschema/#interface">
-<xacro:pioneer_model robot_id="1"  position="2 0 0.3 0 0 0" />
-<xacro:pioneer_model robot_id="2"  position="3 -11 0.3 0 0 0" />
-<xacro:pioneer_model robot_id="3"  position="17 -16 0.3 0 0 -3.1415" />
+<xacro:pioneer_model robot_id="1"  position="1 1 0.3 0 0 0" />
+<xacro:pioneer_model robot_id="2"  position="2 1 0.3 0 0 0" />
+<xacro:pioneer_model robot_id="3"  position="3 1 0.3 0 0 0" />
 </xacro>

File: mrm_sim/models/4robots.xacro (robot description, xacro)
@@ -4,7 +4,7 @@
        xmlns:interface="http://playerstage.sourceforge.net/gazebo/xmlschema/#interface"
        xmlns:xacro="http://playerstage.sourceforge.net/gazebo/xmlschema/#interface">
-<xacro:pioneer_model robot_id="1"  position="2 0 0.3 0 0 0" />
-<xacro:pioneer_model robot_id="2"  position="3 -11 0.3 0 0 0" />
-<xacro:pioneer_model robot_id="3"  position="17 -16 0.3 0 0 -3.1415" />
-<xacro:pioneer_model robot_id="4"  position="3 0 0.3 0 0 0" />
+<xacro:pioneer_model robot_id="1"  position="1 1 0.3 0 0 0" />
+<xacro:pioneer_model robot_id="2"  position="2 1 0.3 0 0 0" />
+<xacro:pioneer_model robot_id="3"  position="3 1 0.3 0 0 0" />
+<xacro:pioneer_model robot_id="4"  position="1 2 0.3 0 0 0" />
 </xacro>

File: mrm_sim/models/5robots.xacro (robot description, xacro)
@@ -4,8 +4,8 @@
        xmlns:interface="http://playerstage.sourceforge.net/gazebo/xmlschema/#interface"
        xmlns:xacro="http://playerstage.sourceforge.net/gazebo/xmlschema/#interface">
-<xacro:pioneer_model robot_id="1"  position="2 0 0.3 0 0 0" />
-<xacro:pioneer_model robot_id="2"  position="3 -11 0.3 0 0 0" />
-<xacro:pioneer_model robot_id="3"  position="17 -16 0.3 0 0 -3.1415" />
-<xacro:pioneer_model robot_id="4"  position="3 0 0.3 0 0 0" />
-<xacro:pioneer_model robot_id="5"  position="4 0 0.3 0 0 0" />
+<xacro:pioneer_model robot_id="1"  position="1 1 0.3 0 0 0" />
+<xacro:pioneer_model robot_id="2"  position="2 1 0.3 0 0 0" />
+<xacro:pioneer_model robot_id="3"  position="3 1 0.3 0 0 0" />
+<xacro:pioneer_model robot_id="4"  position="1 2 0.3 0 0 0" />
+<xacro:pioneer_model robot_id="5"  position="2 2 0.3 0 0 0" />
 </xacro>

File: mrm_sim/models/6robots.xacro (robot description, xacro)
@@ -4,9 +4,9 @@
        xmlns:interface="http://playerstage.sourceforge.net/gazebo/xmlschema/#interface"
        xmlns:xacro="http://playerstage.sourceforge.net/gazebo/xmlschema/#interface">
-<xacro:pioneer_model robot_id="1"  position="2 0 0.3 0 0 0" />
-<xacro:pioneer_model robot_id="2"  position="3 -11 0.3 0 0 0" />
-<xacro:pioneer_model robot_id="3"  position="17 -16 0.3 0 0 -3.1415" />
-<xacro:pioneer_model robot_id="4"  position="3 0 0.3 0 0 0" />
-<xacro:pioneer_model robot_id="5"  position="4 0 0.3 0 0 0" />
-<xacro:pioneer_model robot_id="6"  position="5 0 0.3 0 0 0" />
+<xacro:pioneer_model robot_id="1"  position="1 1 0.3 0 0 0" />
+<xacro:pioneer_model robot_id="2"  position="2 1 0.3 0 0 0" />
+<xacro:pioneer_model robot_id="3"  position="3 1 0.3 0 0 0" />
+<xacro:pioneer_model robot_id="4"  position="1 2 0.3 0 0 0" />
+<xacro:pioneer_model robot_id="5"  position="2 2 0.3 0 0 0" />
+<xacro:pioneer_model robot_id="6"  position="3 2 0.3 0 0 0" />
 </xacro>

File: mrm_sim/models/7robots.xacro (robot description, xacro)
@@ -4,10 +4,10 @@
        xmlns:interface="http://playerstage.sourceforge.net/gazebo/xmlschema/#interface"
        xmlns:xacro="http://playerstage.sourceforge.net/gazebo/xmlschema/#interface">
-<xacro:pioneer_model robot_id="1"  position="2 0 0.3 0 0 0" />
-<xacro:pioneer_model robot_id="2"  position="3 -11 0.3 0 0 0" />
-<xacro:pioneer_model robot_id="3"  position="17 -16 0.3 0 0 -3.1415" />
-<xacro:pioneer_model robot_id="4"  position="3 0 0.3 0 0 0" />
-<xacro:pioneer_model robot_id="5"  position="4 0 0.3 0 0 0" />
-<xacro:pioneer_model robot_id="6"  position="5 0 0.3 0 0 0" />
-<xacro:pioneer_model robot_id="7"  position="6 0 0.3 0 0 0" />
+<xacro:pioneer_model robot_id="1"  position="1 1 0.3 0 0 0" />
+<xacro:pioneer_model robot_id="2"  position="2 1 0.3 0 0 0" />
+<xacro:pioneer_model robot_id="3"  position="3 1 0.3 0 0 0" />
+<xacro:pioneer_model robot_id="4"  position="1 2 0.3 0 0 0" />
+<xacro:pioneer_model robot_id="5"  position="2 2 0.3 0 0 0" />
+<xacro:pioneer_model robot_id="6"  position="3 2 0.3 0 0 0" />
+<xacro:pioneer_model robot_id="7"  position="1 3 0.3 0 0 0" />
 </xacro>

File: mrm_sim/models/8robots.xacro (robot description, xacro)
@@ -4,11 +4,11 @@
        xmlns:interface="http://playerstage.sourceforge.net/gazebo/xmlschema/#interface"
        xmlns:xacro="http://playerstage.sourceforge.net/gazebo/xmlschema/#interface">
-<xacro:pioneer_model robot_id="1"  position="2 0 0.3 0 0 0" />
-<xacro:pioneer_model robot_id="2"  position="3 -11 0.3 0 0 0" />
-<xacro:pioneer_model robot_id="3"  position="17 -16 0.3 0 0 -3.1415" />
-<xacro:pioneer_model robot_id="4"  position="3 0 0.3 0 0 0" />
-<xacro:pioneer_model robot_id="5"  position="4 0 0.3 0 0 0" />
-<xacro:pioneer_model robot_id="6"  position="5 0 0.3 0 0 0" />
-<xacro:pioneer_model robot_id="7"  position="6 0 0.3 0 0 0" />
-<xacro:pioneer_model robot_id="8"  position="7 0 0.3 0 0 0" />
+<xacro:pioneer_model robot_id="1"  position="1 1 0.3 0 0 0" />
+<xacro:pioneer_model robot_id="2"  position="2 1 0.3 0 0 0" />
+<xacro:pioneer_model robot_id="3"  position="3 1 0.3 0 0 0" />
+<xacro:pioneer_model robot_id="4"  position="1 2 0.3 0 0 0" />
+<xacro:pioneer_model robot_id="5"  position="2 2 0.3 0 0 0" />
+<xacro:pioneer_model robot_id="6"  position="3 2 0.3 0 0 0" />
+<xacro:pioneer_model robot_id="7"  position="1 3 0.3 0 0 0" />
+<xacro:pioneer_model robot_id="8"  position="2 3 0.3 0 0 0" />
 </xacro>

File: mrm_sim/models/9robots.xacro (robot description, xacro)
@@ -4,12 +4,12 @@
        xmlns:interface="http://playerstage.sourceforge.net/gazebo/xmlschema/#interface"
        xmlns:xacro="http://playerstage.sourceforge.net/gazebo/xmlschema/#interface">
-<xacro:pioneer_model robot_id="1"  position="2 0 0.3 0 0 0" />
-<xacro:pioneer_model robot_id="2"  position="3 -11 0.3 0 0 0" />
-<xacro:pioneer_model robot_id="3"  position="17 -16 0.3 0 0 -3.1415" />
-<xacro:pioneer_model robot_id="4"  position="3 0 0.3 0 0 0" />
-<xacro:pioneer_model robot_id="5"  position="4 0 0.3 0 0 0" />
-<xacro:pioneer_model robot_id="6"  position="5 0 0.3 0 0 0" />
-<xacro:pioneer_model robot_id="7"  position="6 0 0.3 0 0 0" />
-<xacro:pioneer_model robot_id="8"  position="7 0 0.3 0 0 0" />
-<xacro:pioneer_model robot_id="9"  position="8 0 0.3 0 0 0" />
+<xacro:pioneer_model robot_id="1"  position="1 1 0.3 0 0 0" />
+<xacro:pioneer_model robot_id="2"  position="2 1 0.3 0 0 0" />
+<xacro:pioneer_model robot_id="3"  position="3 1 0.3 0 0 0" />
+<xacro:pioneer_model robot_id="4"  position="1 2 0.3 0 0 0" />
+<xacro:pioneer_model robot_id="5"  position="2 2 0.3 0 0 0" />
+<xacro:pioneer_model robot_id="6"  position="3 2 0.3 0 0 0" />
+<xacro:pioneer_model robot_id="7"  position="1 3 0.3 0 0 0" />
+<xacro:pioneer_model robot_id="8"  position="2 3 0.3 0 0 0" />
+<xacro:pioneer_model robot_id="9"  position="3 3 0.3 0 0 0" />
 </xacro>

File: mrm_sim/models/pioneer_model.xacro (robot description, xacro)
@@ -566,42 +566,45 @@
 	</xacro:macro>
 	<xacro:include filename="$(find mrm_sim)/models/$(arg robots_count)robots.xacro" />
-	<model name='willowgarage'>
-      <static>1</static>
-      <pose>-11 -29 0 0 -0 0</pose>
-      <link name='walls'>
-        <collision name='collision'>
-          <geometry>
-            <mesh>
-              <uri>$(find mrm_sim)/meshes/willowgarage_collision.dae</uri>
-            </mesh>
-          </geometry>
-          <max_contacts>10</max_contacts>
-          <surface>
-            <bounce/>
-            <friction>
-              <ode/>
-            </friction>
-            <contact>
-              <ode/>
-            </contact>
-          </surface>
-        </collision>
-        <visual name='visual'>
-          <geometry>
-            <mesh>
-              <uri>$(find mrm_sim)/meshes/willowgarage_visual.dae</uri>
-            </mesh>
-          </geometry>
-          <cast_shadows>0</cast_shadows>
-        </visual>
-        <velocity_decay>
-          <linear>0</linear>
-          <angular>0</angular>
-        </velocity_decay>
-        <self_collide>0</self_collide>
-        <kinematic>0</kinematic>
-        <gravity>1</gravity>
-      </link>
-    </model>
+  <model name="willow_closed">
+    <static>true</static>
+    <pose>0 0 0.001 0 0 0</pose>
+    <link name="walls">
+      <collision name="collision">
+        <geometry>
+          <mesh>
+	    <uri>$(find mrm_sim)/meshes/office_mesh/willowgarage_collision.dae</uri>
+          </mesh>
+        </geometry>
+	<max_contacts>100</max_contacts>
+        <surface>
+          <friction>
+            <ode>
+              <mu>0.99</mu>
+              <mu2>0.99</mu2>
+            </ode>
+          </friction>
+          <bounce/>
+          <contact>
+            <ode/>
+          </contact>
+        </surface>
+      </collision>
+      <visual name="visual">
+        <geometry>
+          <mesh>
+           <uri>$(find mrm_sim)/meshes/office_mesh/willowgarage_visual.dae</uri>
+          </mesh>
+        </geometry>
+        <cast_shadows>true</cast_shadows>
+      </visual>
+      <velocity_decay>
+	<linear>0</linear>
+	<angular>0</angular>
+      </velocity_decay>
+      <self_collide>0</self_collide>
+      <kinematic>0</kinematic>
+      <gravity>1</gravity>
+    </link>
+  </model>
   </world>
 </sdf>
