Commit message: Updated lidar (fixed error in xacro)

File: mrm_sim/models/10robots.xacro (robot description, xacro)
@@ -4,13 +4,13 @@
        xmlns:interface="http://playerstage.sourceforge.net/gazebo/xmlschema/#interface"
        xmlns:xacro="http://playerstage.sourceforge.net/gazebo/xmlschema/#interface">
-<xacro:pioneer_model robot_id="1"  position="1 1 0.3 0 0 0" />
-<xacro:pioneer_model robot_id="2"  position="2 1 0.3 0 0 0" />
-<xacro:pioneer_model robot_id="3"  position="3 1 0.3 0 0 0" />
-<xacro:pioneer_model robot_id="4"  position="1 2 0.3 0 0 0" />
-<xacro:pioneer_model robot_id="5"  position="2 2 0.3 0 0 0" />
-<xacro:pioneer_model robot_id="6"  position="3 2 0.3 0 0 0" />
-<xacro:pioneer_model robot_id="7"  position="1 3 0.3 0 0 0" />
-<xacro:pioneer_model robot_id="8"  position="2 3 0.3 0 0 0" />
-<xacro:pioneer_model robot_id="9"  position="3 3 0.3 0 0 0" />
-<xacro:pioneer_model robot_id="10" position="4 1 0.3 0 0 0" />
+<xacro:hamster_model robot_id="1"  position="1 1 0.3 0 0 0" />
+<xacro:hamster_model robot_id="2"  position="2 1 0.3 0 0 0" />
+<xacro:hamster_model robot_id="3"  position="3 1 0.3 0 0 0" />
+<xacro:hamster_model robot_id="4"  position="1 2 0.3 0 0 0" />
+<xacro:hamster_model robot_id="5"  position="2 2 0.3 0 0 0" />
+<xacro:hamster_model robot_id="6"  position="3 2 0.3 0 0 0" />
+<xacro:hamster_model robot_id="7"  position="1 3 0.3 0 0 0" />
+<xacro:hamster_model robot_id="8"  position="2 3 0.3 0 0 0" />
+<xacro:hamster_model robot_id="9"  position="3 3 0.3 0 0 0" />
+<xacro:hamster_model robot_id="10" position="4 1 0.3 0 0 0" />
 </xacro>

File: mrm_sim/models/1robots.xacro (robot description, xacro)
@@ -4,4 +4,4 @@
        xmlns:interface="http://playerstage.sourceforge.net/gazebo/xmlschema/#interface"
        xmlns:xacro="http://playerstage.sourceforge.net/gazebo/xmlschema/#interface">
-<xacro:pioneer_model robot_id="1"  position="1 1 0.3 0 0 0" />
+<xacro:hamster_model robot_id="1"  position="1 1 0.3 0 0 0" />
 </xacro>

File: mrm_sim/models/2robots.xacro (robot description, xacro)
@@ -4,5 +4,5 @@
        xmlns:interface="http://playerstage.sourceforge.net/gazebo/xmlschema/#interface"
        xmlns:xacro="http://playerstage.sourceforge.net/gazebo/xmlschema/#interface">
-<xacro:pioneer_model robot_id="1"  position="1 1 0.3 0 0 0" />
-<xacro:pioneer_model robot_id="2"  position="2 1 0.3 0 0 0" />
+<xacro:hamster_model robot_id="1"  position="1 1 0.3 0 0 0" />
+<xacro:hamster_model robot_id="2"  position="2 1 0.3 0 0 0" />
 </xacro>

File: mrm_sim/models/3robots.xacro (robot description, xacro)
@@ -4,6 +4,6 @@
        xmlns:interface="http://playerstage.sourceforge.net/gazebo/xmlschema/#interface"
        xmlns:xacro="http://playerstage.sourceforge.net/gazebo/xmlschema/#interface">
-<xacro:pioneer_model robot_id="1"  position="1 1 0.3 0 0 0" />
-<xacro:pioneer_model robot_id="2"  position="2 1 0.3 0 0 0" />
-<xacro:pioneer_model robot_id="3"  position="3 1 0.3 0 0 0" />
+<xacro:hamster_model robot_id="1"  position="1 1 0.3 0 0 0" />
+<xacro:hamster_model robot_id="2"  position="2 1 0.3 0 0 0" />
+<xacro:hamster_model robot_id="3"  position="3 1 0.3 0 0 0" />
 </xacro>

File: mrm_sim/models/4robots.xacro (robot description, xacro)
@@ -4,7 +4,7 @@
        xmlns:interface="http://playerstage.sourceforge.net/gazebo/xmlschema/#interface"
        xmlns:xacro="http://playerstage.sourceforge.net/gazebo/xmlschema/#interface">
-<xacro:pioneer_model robot_id="1"  position="1 1 0.3 0 0 0" />
-<xacro:pioneer_model robot_id="2"  position="2 1 0.3 0 0 0" />
-<xacro:pioneer_model robot_id="3"  position="3 1 0.3 0 0 0" />
-<xacro:pioneer_model robot_id="4"  position="1 2 0.3 0 0 0" />
+<xacro:hamster_model robot_id="1"  position="1 1 0.3 0 0 0" />
+<xacro:hamster_model robot_id="2"  position="2 1 0.3 0 0 0" />
+<xacro:hamster_model robot_id="3"  position="3 1 0.3 0 0 0" />
+<xacro:hamster_model robot_id="4"  position="1 2 0.3 0 0 0" />
 </xacro>

File: mrm_sim/models/5robots.xacro (robot description, xacro)
@@ -4,8 +4,8 @@
        xmlns:interface="http://playerstage.sourceforge.net/gazebo/xmlschema/#interface"
        xmlns:xacro="http://playerstage.sourceforge.net/gazebo/xmlschema/#interface">
-<xacro:pioneer_model robot_id="1"  position="1 1 0.3 0 0 0" />
-<xacro:pioneer_model robot_id="2"  position="2 1 0.3 0 0 0" />
-<xacro:pioneer_model robot_id="3"  position="3 1 0.3 0 0 0" />
-<xacro:pioneer_model robot_id="4"  position="1 2 0.3 0 0 0" />
-<xacro:pioneer_model robot_id="5"  position="2 2 0.3 0 0 0" />
+<xacro:hamster_model robot_id="1"  position="1 1 0.3 0 0 0" />
+<xacro:hamster_model robot_id="2"  position="2 1 0.3 0 0 0" />
+<xacro:hamster_model robot_id="3"  position="3 1 0.3 0 0 0" />
+<xacro:hamster_model robot_id="4"  position="1 2 0.3 0 0 0" />
+<xacro:hamster_model robot_id="5"  position="2 2 0.3 0 0 0" />
 </xacro>

File: mrm_sim/models/6robots.xacro (robot description, xacro)
@@ -4,9 +4,9 @@
        xmlns:interface="http://playerstage.sourceforge.net/gazebo/xmlschema/#interface"
        xmlns:xacro="http://playerstage.sourceforge.net/gazebo/xmlschema/#interface">
-<xacro:pioneer_model robot_id="1"  position="1 1 0.3 0 0 0" />
-<xacro:pioneer_model robot_id="2"  position="2 1 0.3 0 0 0" />
-<xacro:pioneer_model robot_id="3"  position="3 1 0.3 0 0 0" />
-<xacro:pioneer_model robot_id="4"  position="1 2 0.3 0 0 0" />
-<xacro:pioneer_model robot_id="5"  position="2 2 0.3 0 0 0" />
-<xacro:pioneer_model robot_id="6"  position="3 2 0.3 0 0 0" />
+<xacro:hamster_model robot_id="1"  position="1 1 0.3 0 0 0" />
+<xacro:hamster_model robot_id="2"  position="2 1 0.3 0 0 0" />
+<xacro:hamster_model robot_id="3"  position="3 1 0.3 0 0 0" />
+<xacro:hamster_model robot_id="4"  position="1 2 0.3 0 0 0" />
+<xacro:hamster_model robot_id="5"  position="2 2 0.3 0 0 0" />
+<xacro:hamster_model robot_id="6"  position="3 2 0.3 0 0 0" />
 </xacro>

File: mrm_sim/models/7robots.xacro (robot description, xacro)
@@ -4,10 +4,10 @@
        xmlns:interface="http://playerstage.sourceforge.net/gazebo/xmlschema/#interface"
        xmlns:xacro="http://playerstage.sourceforge.net/gazebo/xmlschema/#interface">
-<xacro:pioneer_model robot_id="1"  position="1 1 0.3 0 0 0" />
-<xacro:pioneer_model robot_id="2"  position="2 1 0.3 0 0 0" />
-<xacro:pioneer_model robot_id="3"  position="3 1 0.3 0 0 0" />
-<xacro:pioneer_model robot_id="4"  position="1 2 0.3 0 0 0" />
-<xacro:pioneer_model robot_id="5"  position="2 2 0.3 0 0 0" />
-<xacro:pioneer_model robot_id="6"  position="3 2 0.3 0 0 0" />
-<xacro:pioneer_model robot_id="7"  position="1 3 0.3 0 0 0" />
+<xacro:hamster_model robot_id="1"  position="1 1 0.3 0 0 0" />
+<xacro:hamster_model robot_id="2"  position="2 1 0.3 0 0 0" />
+<xacro:hamster_model robot_id="3"  position="3 1 0.3 0 0 0" />
+<xacro:hamster_model robot_id="4"  position="1 2 0.3 0 0 0" />
+<xacro:hamster_model robot_id="5"  position="2 2 0.3 0 0 0" />
+<xacro:hamster_model robot_id="6"  position="3 2 0.3 0 0 0" />
+<xacro:hamster_model robot_id="7"  position="1 3 0.3 0 0 0" />
 </xacro>

File: mrm_sim/models/8robots.xacro (robot description, xacro)
@@ -4,11 +4,11 @@
        xmlns:interface="http://playerstage.sourceforge.net/gazebo/xmlschema/#interface"
        xmlns:xacro="http://playerstage.sourceforge.net/gazebo/xmlschema/#interface">
-<xacro:pioneer_model robot_id="1"  position="1 1 0.3 0 0 0" />
-<xacro:pioneer_model robot_id="2"  position="2 1 0.3 0 0 0" />
-<xacro:pioneer_model robot_id="3"  position="3 1 0.3 0 0 0" />
-<xacro:pioneer_model robot_id="4"  position="1 2 0.3 0 0 0" />
-<xacro:pioneer_model robot_id="5"  position="2 2 0.3 0 0 0" />
-<xacro:pioneer_model robot_id="6"  position="3 2 0.3 0 0 0" />
-<xacro:pioneer_model robot_id="7"  position="1 3 0.3 0 0 0" />
-<xacro:pioneer_model robot_id="8"  position="2 3 0.3 0 0 0" />
+<xacro:hamster_model robot_id="1"  position="1 1 0.3 0 0 0" />
+<xacro:hamster_model robot_id="2"  position="2 1 0.3 0 0 0" />
+<xacro:hamster_model robot_id="3"  position="3 1 0.3 0 0 0" />
+<xacro:hamster_model robot_id="4"  position="1 2 0.3 0 0 0" />
+<xacro:hamster_model robot_id="5"  position="2 2 0.3 0 0 0" />
+<xacro:hamster_model robot_id="6"  position="3 2 0.3 0 0 0" />
+<xacro:hamster_model robot_id="7"  position="1 3 0.3 0 0 0" />
+<xacro:hamster_model robot_id="8"  position="2 3 0.3 0 0 0" />
 </xacro>

File: mrm_sim/models/9robots.xacro (robot description, xacro)
@@ -4,12 +4,12 @@
        xmlns:interface="http://playerstage.sourceforge.net/gazebo/xmlschema/#interface"
        xmlns:xacro="http://playerstage.sourceforge.net/gazebo/xmlschema/#interface">
-<xacro:pioneer_model robot_id="1"  position="1 1 0.3 0 0 0" />
-<xacro:pioneer_model robot_id="2"  position="2 1 0.3 0 0 0" />
-<xacro:pioneer_model robot_id="3"  position="3 1 0.3 0 0 0" />
-<xacro:pioneer_model robot_id="4"  position="1 2 0.3 0 0 0" />
-<xacro:pioneer_model robot_id="5"  position="2 2 0.3 0 0 0" />
-<xacro:pioneer_model robot_id="6"  position="3 2 0.3 0 0 0" />
-<xacro:pioneer_model robot_id="7"  position="1 3 0.3 0 0 0" />
-<xacro:pioneer_model robot_id="8"  position="2 3 0.3 0 0 0" />
-<xacro:pioneer_model robot_id="9"  position="3 3 0.3 0 0 0" />
+<xacro:hamster_model robot_id="1"  position="1 1 0.3 0 0 0" />
+<xacro:hamster_model robot_id="2"  position="2 1 0.3 0 0 0" />
+<xacro:hamster_model robot_id="3"  position="3 1 0.3 0 0 0" />
+<xacro:hamster_model robot_id="4"  position="1 2 0.3 0 0 0" />
+<xacro:hamster_model robot_id="5"  position="2 2 0.3 0 0 0" />
+<xacro:hamster_model robot_id="6"  position="3 2 0.3 0 0 0" />
+<xacro:hamster_model robot_id="7"  position="1 3 0.3 0 0 0" />
+<xacro:hamster_model robot_id="8"  position="2 3 0.3 0 0 0" />
+<xacro:hamster_model robot_id="9"  position="3 3 0.3 0 0 0" />
 </xacro>

File: mrm_sim/models/pioneer_model.xacro (robot description, xacro)
@@ -77,6 +77,6 @@
       <shadows>1</shadows>
     </scene>
-    <xacro:macro name="pioneer_model" params="robot_id position">
-	    <model name='pioneer3at_${robot_id}'>
+    <xacro:macro name="hamster_model" params="robot_id position">
+	    <model name='hamster3at_${robot_id}'>
     	  <pose>${position}</pose>
 	      <!-- Shaft #1 -->
@@ -386,4 +386,96 @@
 	        <kinematic>0</kinematic>
 	        <gravity>1</gravity>
+	      </link>
+	      <link name="rplidar_link">
+		<pose>-0.045 0 0.095 0 0 0</pose>
+		<visual name="visual">
+		  <geometry>
+		    <cylinder>
+		      <radius>0.035</radius>
+		      <length>0.02</length>
+		    </cylinder>
+		  </geometry>
+		</visual>
+		<collision name="collision">
+		  <geometry>
+		    <cylinder>
+		      <radius>0.035</radius>
+		      <length>0.02</length>
+		    </cylinder>
+		  </geometry>
+		</collision>
+		<sensor name="rplidar" type="ray">
+		  <ray>
+		    <scan>
+		      <horizontal>
+			<samples>360</samples>
+			<resolution>1</resolution>
+			<min_angle>-3.1415</min_angle>
+			<max_angle>3.1415</max_angle>
+		      </horizontal>
+		    </scan>
+		    <range>
+		      <min>0.10</min>
+		      <max>6</max>
+		      <resolution>0.01</resolution>
+		    </range>
+		    <noise>
+		      <type>gaussian</type>
+		      <mean>0.0</mean>
+		      <stddev>0.01</stddev>
+		    </noise>
+		  </ray>
+		  <plugin name="laser" filename="libRayPlugin.so" />
+		  <always_on>1</always_on>
+		  <update_rate>6</update_rate>
+		  <visualize>false</visualize>
+		  <plugin name="gazebo_ros_laser_controller" filename="libgazebo_ros_laser.so">
+		    <gaussianNoise>0.005</gaussianNoise>
+		    <alwaysOn>true</alwaysOn>
+		    <updateRate>6</updateRate>
+		    <topicName>/hamster_${robot_id}/scan_rplidar</topicName>
+		    <frameName>/hamster_${robot_id}/rplidar_link</frameName>
+		    <hokuyoMinIntensity>101</hokuyoMinIntensity>
+		  </plugin>
+		</sensor>
+	      </link>
+	      <link name="camera::link">
+		<pose>0.10 0.05 0.15 0 0 0</pose>
+		<inertial>
+		  <mass>0.1</mass>
+		</inertial>
+		<collision name="collision">
+		  <geometry>
+		    <box>
+		      <size>0.01 0.01 0.01</size>
+		    </box>
+		  </geometry>
+		</collision>
+		<visual name="visual">
+		  <geometry>
+		    <box>
+		      <size>0.01 0.01 0.01</size>
+		    </box>
+		  </geometry>
+		</visual>
+		<sensor name="camera" type="camera">
+		  <camera>
+		    <horizontal_fov>0.752</horizontal_fov>
+		    <image>
+		      <width>640</width>
+		      <height>480</height>
+		    </image>
+		    <clip>
+		      <near>0.1</near>
+		      <far>100</far>
+		    </clip>
+		  </camera>
+		  <always_on>1</always_on>
+		  <update_rate>15</update_rate>
+		  <visualize>false</visualize>
+		  <plugin name='ros_camera' filename='libgazebo_ros_camera.so'>
+			  <robotNamespace>/hamster_${robot_id}</robotNamespace>
+		  </plugin>
+		</sensor>
 	      </link>
 	      <joint name='shell_to_chassis' type='revolute'>
@@ -447,149 +539,18 @@
 	        </axis>
 	      </joint>
-	      <link name='hokuyo::link'>
-	        <inertial>
-	          <mass>0.1</mass>
-	          <inertia>
-	            <ixx>1</ixx>
-	            <ixy>0</ixy>
-	            <ixz>0</ixz>
-	            <iyy>1</iyy>
-	            <iyz>0</iyz>
-	            <izz>1</izz>
-	          </inertia>
-	        </inertial>
-	        <visual name='visual'>
-	          <geometry>
-	            <mesh filename="package://mrm_sim/meshes/hokuyo.dae" />
-	          </geometry>
-	        </visual>
-	        <collision name='collision-base'>
-	          <pose>0 0 -0.0145 0 -0 0</pose>
-	          <geometry>
-	            <box>
-	              <size>0.05 0.05 0.041</size>
-	            </box>
-	          </geometry>
-	          <max_contacts>10</max_contacts>
-	          <surface>
-	            <bounce/>
-	            <friction>
-	              <ode/>
-	            </friction>
-	            <contact>
-	              <ode/>
-	            </contact>
-	          </surface>
-	        </collision>
-	        <collision name='collision-top'>
-	          <pose>0 0 0.0205 0 -0 0</pose>
-	          <geometry>
-	            <cylinder>
-	              <radius>0.021</radius>
-	              <length>0.029</length>
-	            </cylinder>
-	          </geometry>
-	          <max_contacts>10</max_contacts>
-	          <surface>
-	            <bounce/>
-	            <friction>
-	              <ode/>
-	            </friction>
-	            <contact>
-	              <ode/>
-	            </contact>
-	          </surface>
-	        </collision>
-	        <sensor name='laser' type='ray'>
-	          <pose>0 0 0 0 -0 0</pose>
-	          <ray>
-	            <scan>
-	              <horizontal>
-	                <samples>1040</samples>
-	                <resolution>1</resolution>
-	                <min_angle>-2.26889</min_angle>
-	                <max_angle>2.2689</max_angle>
-	              </horizontal>
-	            </scan>
-	            <range>
-	              <min>0.1</min>
-	              <max>30</max>
-	              <resolution>0.01</resolution>
-	            </range>
-	          </ray>
-	          <!-- <plugin name='laser' filename='libRayPlugin.so'/> -->
-	          <plugin name='gazebo_ros_hokuyo_laser_controller' filename='libgazebo_ros_laser.so'>
-	            <gaussianNoise>0.01</gaussianNoise>
-	            <alwaysOn>true</alwaysOn>
-	            <hokuyoMinIntensity>101</hokuyoMinIntensity>
-	            <updateRate>40.0</updateRate>
-	            <topicName>/pioneer_${robot_id}/scan_raw</topicName>
-	            <frameName>/pioneer_${robot_id}/odom_tf__not_used__a</frameName>
-	            <interface:laser/>
-	          </plugin>
-	          <always_on>1</always_on>
-	          <update_rate>30</update_rate>
-	          <visualize>1</visualize>
-	        </sensor>
-	        <velocity_decay>
-	          <linear>0</linear>
-	          <angular>0</angular>
-	        </velocity_decay>
-	        <pose>$(arg laser_forward_offset) 0 0.06 0 -0 0</pose>
-	        <self_collide>0</self_collide>
-	        <kinematic>0</kinematic>
-	        <gravity>1</gravity>
-	      </link>
-	      <joint name='hokuyo_joint' type='revolute'>
-	        <child>hokuyo::link</child>
-	        <parent>chassis</parent>
-	        <axis>
-	          <xyz>0 0 1</xyz>
-	          <limit>
-	            <upper>0</upper>
-	            <lower>0</lower>
-	          </limit>
-	        </axis>
+	      <joint name="rplidar_to_chassis" type="revolute">
+		<pose>0 0 0 0 0 0</pose>
+		<child>rplidar_link</child>
+		<parent>chassis</parent>
+		<axis>
+		  <xyz>0 0 1</xyz>
+		  <limit>
+		    <upper>0</upper>
+		    <lower>0</lower>
+		  </limit>
+		</axis>
 	      </joint>
-		    <link name="camera::link">
-		      <pose>0.10 0.05 0.15 0 0 0</pose>
-		      <inertial>
-		        <mass>0.1</mass>
-		      </inertial>
-		      <collision name="collision">
-		        <geometry>
-		          <box>
-		            <size>0.1 0.1 0.1</size>
-		          </box>
-		        </geometry>
-		      </collision>
-		      <visual name="visual">
-		        <geometry>
-		          <box>
-		            <size>0.1 0.1 0.1</size>
-		          </box>
-		        </geometry>
-		      </visual>
-		      <sensor name="camera" type="camera">
-		        <camera>
-		          <horizontal_fov>0.752</horizontal_fov>
-		          <image>
-		            <width>640</width>
-		            <height>480</height>
-		          </image>
-		          <clip>
-		            <near>0.1</near>
-		            <far>100</far>
-		          </clip>
-		        </camera>
-		        <always_on>1</always_on>
-		        <update_rate>15</update_rate>
-		        <visualize>false</visualize>
-		        <plugin name='ros_camera' filename='libgazebo_ros_camera.so'>
-	        		<robotNamespace>/pioneer_${robot_id}</robotNamespace>
-		        </plugin>
-		      </sensor>
-		    </link>
 	      <joint name="camera_joint" type="revolute">
+		<pose>0 0 0 0 0 0</pose>
 	        <child>camera::link</child>
 	        <parent>chassis</parent>
@@ -604,5 +565,5 @@
 	      <plugin name='skid_steer_drive_controller' filename='libgazebo_ros_skid_steer_drive.so'>
 	        <updateRate>100.0</updateRate>
-	        <robotNamespace>/pioneer_${robot_id}</robotNamespace>
+	        <robotNamespace>/hamster_${robot_id}</robotNamespace>
 	        <leftFrontJoint>left_front</leftFrontJoint>
 	        <rightFrontJoint>right_front</rightFrontJoint>
@@ -612,5 +573,5 @@
 	        <wheelDiameter>0.215</wheelDiameter>
 	        <odometryTopic>odom_raw</odometryTopic>
-	        <robotBaseFrame>/pioneer_${robot_id}/odom_tf</robotBaseFrame>
+	        <robotBaseFrame>/hamster_${robot_id}/odom_tf</robotBaseFrame>
 	        <torque>120</torque>
 	        <commandTopic>cmd_vel</commandTopic>
@@ -619,5 +580,5 @@
 <!-- 	      <plugin filename="libgazebo_ros_imu.so" name="imu_en_ros">
 	  		  <bodyName>chassis</bodyName>
-	  		  <robotNamespace>/pioneer_${robot_id}</robotNamespace>
+	  		  <robotNamespace>/hamster_${robot_id}</robotNamespace>
 	  		  <topicName>imu</topicName>
 	  		  <gaussianNoise>0.00</gaussianNoise>
