Commit message: Updated model to look closer to real hamster (in work)

File: mrm_sim/models/pioneer_model.xacro (robot description, xacro)
@@ -104,5 +104,5 @@
 	          <geometry>
 	            <box>
-	              <size>0.501 0.2 0.19</size>
+	              <size>0.185 0.1 0.03</size>
 	            </box>
 	          </geometry>
@@ -120,7 +120,10 @@
 	        <visual name='visual'>
 	          <geometry>
-	            <mesh>
+<!--	            <mesh>
 	              <uri>$(find mrm_sim)/meshes/chassis.dae</uri>
-	            </mesh>
+	            </mesh>-->
+		    <box>
+	              <size>0.185 0.1 0.03</size>
+	            </box>
 	          </geometry>
 	        </visual>
@@ -134,10 +137,10 @@
 	      </link>
 	      <link name='right_front_wheel'>
-	        <pose>0.125 -0.1005 -0.06 1.5707 -0 0</pose>
+	        <pose>0.083 -0.0725 -0.005 1.5707 -0 0</pose>
 	        <collision name='collision'>
 	          <geometry>
 	            <cylinder>
-	              <radius>0.11</radius>
-	              <length>0.075</length>
+	              <radius>0.035</radius>
+	              <length>0.035</length>
 	            </cylinder>
 	          </geometry>
@@ -161,4 +164,5 @@
 	          <geometry>
 	            <mesh>
+		      <scale>0.318 0.318 0.35</scale>
 	              <uri>$(find mrm_sim)/meshes/wheel.dae</uri>
 	            </mesh>
@@ -185,10 +189,10 @@
 	      </link>
 	      <link name='left_front_wheel'>
-	        <pose>0.125 0.1005 -0.06 1.5707 -0 0</pose>
+	        <pose>0.083 0.0725 -0.005 1.5707 -0 0</pose>
 	        <collision name='collision'>
 	          <geometry>
 	            <cylinder>
-	              <radius>0.11</radius>
-	              <length>0.075</length>
+	              <radius>0.035</radius>
+	              <length>0.035</length>
 	            </cylinder>
 	          </geometry>
@@ -212,4 +216,5 @@
 	          <geometry>
 	            <mesh>
+		      <scale>0.318 0.318 0.35</scale>
 	              <uri>$(find mrm_sim)/meshes/wheel.dae</uri>
 	            </mesh>
@@ -236,10 +241,10 @@
 	      </link>
 	      <link name='right_rear_wheel'>
-	        <pose>-0.125 -0.1005 -0.06 1.5707 -0 0</pose>
+	        <pose>-0.083 -0.0725 -0.005 1.5707 -0 0</pose>
 	        <collision name='collision'>
 	          <geometry>
 	            <cylinder>
-	              <radius>0.11</radius>
-	              <length>0.075</length>
+	              <radius>0.035</radius>
+	              <length>0.035</length>
 	            </cylinder>
 	          </geometry>
@@ -263,4 +268,5 @@
 	          <geometry>
 	            <mesh>
+		      <scale>0.318 0.318 0.35</scale>
 	              <uri>$(find mrm_sim)/meshes/wheel.dae</uri>
 	            </mesh>
@@ -287,10 +293,10 @@
 	      </link>
 	      <link name='left_rear_wheel'>
-	        <pose>-0.125 0.1005 -0.06 1.5707 -0 0</pose>
+	        <pose>-0.083 0.0725 -0.005 1.5707 -0 0</pose>
 	        <collision name='collision'>
 	          <geometry>
 	            <cylinder>
-	              <radius>0.11</radius>
-	              <length>0.075</length>
+	              <radius>0.035</radius>
+	              <length>0.035</length>
 	            </cylinder>
 	          </geometry>
@@ -314,5 +320,5 @@
 	          <geometry>
 	            <mesh>
-	              <scale>1 1 1</scale>
+	              <scale>0.318 0.318 0.35</scale>
 	              <uri>$(find mrm_sim)/meshes/wheel.dae</uri>
 	            </mesh>

Commit message: Added hamster shell

File: mrm_sim/models/pioneer_model.xacro (robot description, xacro)
@@ -104,5 +104,5 @@
 	          <geometry>
 	            <box>
-	              <size>0.185 0.1 0.03</size>
+	              <size>0.185 0.1 0.02</size>
 	            </box>
 	          </geometry>
@@ -120,10 +120,53 @@
 	        <visual name='visual'>
 	          <geometry>
-<!--	            <mesh>
-	              <uri>$(find mrm_sim)/meshes/chassis.dae</uri>
-	            </mesh>-->
 		    <box>
 	              <size>0.185 0.1 0.03</size>
 	            </box>
+	          </geometry>
+	        </visual>
+	        <velocity_decay>
+	          <linear>0</linear>
+	          <angular>0</angular>
+	        </velocity_decay>
+	        <self_collide>0</self_collide>
+	        <kinematic>0</kinematic>
+	        <gravity>1</gravity>
+	      </link>
+	      <link name='shell'>
+		<pose>0.005 0 -0.01 0 0 0</pose>
+	        <inertial>
+	          <mass>1</mass>
+	          <inertia>
+	            <ixx>0.3338</ixx>
+	            <ixy>0</ixy>
+	            <ixz>0</ixz>
+	            <iyy>0.4783</iyy>
+	            <iyz>0</iyz>
+	            <izz>0.3338</izz>
+	          </inertia>
+	        </inertial>
+	        <collision name='collision'>
+	          <geometry>
+		    <box>
+	              <size>0.25 0.2 0.08</size>
+	            </box>
+		  </geometry>
+	          <max_contacts>10</max_contacts>
+	          <surface>
+	            <bounce/>
+	            <friction>
+	              <ode/>
+	            </friction>
+	            <contact>
+	              <ode/>
+	            </contact>
+	          </surface>
+	        </collision>
+	        <visual name='visual'>
+	          <geometry>
+	            <mesh>
+		      <scale>1 1 1</scale>
+	              <uri>$(find mrm_sim)/meshes/shell.dae</uri>
+	            </mesh>
 	          </geometry>
 	        </visual>
@@ -344,4 +387,16 @@
 	        <gravity>1</gravity>
 	      </link>
+	      <joint name='shell_to_chassis' type='revolute'>
+	        <pose>0 0 0 0 0 0</pose>
+	        <child>shell</child>
+	        <parent>chassis</parent>
+	        <axis>
+	          <xyz>0 1 0</xyz>
+	          <limit>
+	            <lower>0</lower>
+	            <upper>0</upper>
+	          </limit>
+	        </axis>
+	      </joint>
 	      <joint name='right_front' type='revolute'>
 	        <pose>0 0 0 0 -0 0</pose>

Commit message: Tested /cmd_vel msgs control. All works

File: mrm_sim/models/pioneer_model.xacro (robot description, xacro)
@@ -148,7 +148,8 @@
 	        <collision name='collision'>
 	          <geometry>
-		    <box>
-	              <size>0.25 0.2 0.08</size>
-	            </box>
+	            <mesh>
+		      <scale>1 1 1</scale>
+	              <uri>$(find mrm_sim)/meshes/shell.dae</uri>
+	            </mesh>
 		  </geometry>
 	          <max_contacts>10</max_contacts>
@@ -574,5 +575,5 @@
 	        <odometryTopic>odom_raw</odometryTopic>
 	        <robotBaseFrame>/hamster_${robot_id}/odom_tf</robotBaseFrame>
-	        <torque>120</torque>
+	        <torque>30</torque>
 	        <commandTopic>cmd_vel</commandTopic>
 	        <broadcastTF>1</broadcastTF>
